Commit message: base rl_files added

File: catbot_description/urdf/bot.xacro (robot description, xacro)
@@ -2,5 +2,5 @@
 <robot name="catbot" xmlns:xacro="http://www.ros.org/wiki/xacro">
 <xacro:include filename="$(find catbot_description)/urdf/main.gazebo" />
-<!-- <link name="base_footprint">
+<link name="base_footprint">
 <inertial>
     <origin xyz="0.0 0.0 0.0" rpy="0 0 0" />
@@ -20,5 +20,5 @@
     </geometry>
 </collision>
-</link> -->
+</link>
 <link name="base_body">
 <inertial>
@@ -40,10 +40,10 @@
 </collision>
 </link>
-<!-- <joint name="base_joint" type="fixed">
+<joint name="base_joint" type="fixed">
     <axis xyz="0 0 0" />
-    <origin xyz="0 0 0.75" rpy="0 0 0" />
+    <origin xyz="0 0 0.80" rpy="0 0 0" />
     <parent link="base_footprint" />
     <child link="base_body" />
-</joint> -->
+</joint>
 <!-- ##########################################################
      ######################### left leg ########################

Commit message: stable standing pose added

File: catbot_description/urdf/bot.xacro (robot description, xacro)
@@ -23,7 +23,7 @@
 <link name="base_body">
 <inertial>
-    <origin xyz="0.0 0.0 0.0" rpy="0 0 0" />
-    <mass value="0.5" />
-    <inertia ixx="0.1" ixy="0.1" ixz="0.1" iyy="0.1" iyz="0.1" izz="0.1"/>
+    <origin xyz="0.0 0.0 0.5" rpy="0 0 0" />
+    <mass value="4.0" />
+    <inertia ixx="0.42841" ixy="-2.3739" ixz="0.00227" iyy="0.43178" iyz="1.46390" izz="0.08742"/>
 </inertial>
 <visual>
@@ -51,5 +51,5 @@
 <joint
     name="bum_zlj" type="revolute">
-    <origin xyz="-0.02 0.265 0.16" rpy="0 0 0" />
+    <origin xyz="-0.02 0.265 0.16" rpy="0 -0.3 0" />
     <parent link="base_body" />
     <child link="bum_zl" />
@@ -60,5 +60,5 @@
 <link name="bum_zl">
 <inertial>
-    <origin xyz="0.0 0.0 0.0" rpy="0 0 0" />
+    <origin xyz="0.0 0.0 -0.19" rpy="0 0 0" />
     <mass value="0.3" />
     <inertia ixx="0.1" ixy="0.1" ixz="0.1" iyy="0.1" iyz="0.1" izz="0.1"/>
@@ -88,5 +88,5 @@
 <link name="bum_xl">
 <inertial>
-    <origin xyz="0.0 0.0 0.0" rpy="0 0 0" />
+    <origin xyz="0.0 0.0 -0.19" rpy="0 0 0" />
     <mass value="0.3" />
     <inertia ixx="0.1" ixy="0.1" ixz="0.1" iyy="0.1" iyz="0.1" izz="0.1"/>
@@ -107,4 +107,5 @@
 <joint
     name="bum_ylj" type="revolute">
+    <!-- <origin xyz="0 0 0" rpy="0 0.35 3.142" /> -->
     <origin xyz="0 0 0" rpy="0 0 3.142" />
     <parent link="bum_xl" />
@@ -116,7 +117,7 @@
 <link name="left_hip">
 <inertial>
-    <origin xyz="0.0 0.0 0.0" rpy="0 0 0" />
-    <mass value="0.3" />
-    <inertia ixx="0.1" ixy="0.1" ixz="0.1" iyy="0.1" iyz="0.1" izz="0.1"/>
+    <origin xyz="0.0 0 -0.19" rpy="0 0 0" />
+    <mass value="0.3" />
+    <inertia ixx="0.31319" ixy="-1.5919" ixz="0.00039" iyy="0.314057" iyz="-0.00060" izz="0.02458"/>
 </inertial>
 <visual>
@@ -135,5 +136,5 @@
 <joint
     name="knee_left" type="revolute">
-    <origin xyz="0 0 -0.335" rpy="0 0 0" />
+    <origin xyz="0 0 -0.335" rpy="0 -0.5 0" />
     <parent link="left_hip" />
     <child link="left_shin" />
@@ -144,7 +145,7 @@
 <link name="left_shin">
 <inertial>
-    <origin xyz="0.0 0.0 0.0" rpy="0 0 0" />
-    <mass value="0.3" />
-    <inertia ixx="0.1" ixy="0.1" ixz="0.1" iyy="0.1" iyz="0.1" izz="0.1"/>
+    <origin xyz="0.0 0.0 -0.2" rpy="0 0 0" />
+    <mass value="0.3" />
+    <inertia ixx="0.283162" ixy="0.00034" ixz="0.001493" iyy="0.284290" iyz="0.000595" izz="0.0277465"/>
 </inertial>
 <visual>
@@ -163,9 +164,9 @@
 <joint
     name="ankle_lj" type="revolute">
-    <origin xyz="0 0 -0.58" rpy="0 0 0" />
+    <origin xyz="0 0 -0.58" rpy="0 0.3 0" />
     <parent link="left_shin" />
     <child link="left_ankle" />
     <axis xyz="0 1 0" />
-    <limit lower="-1.3" upper="0" effort="150.0" velocity="3"/>
+    <limit lower="-1.3" upper="0.3" effort="150.0" velocity="3"/>
     <!-- dynamics damping="5" friction="0.0"/ -->
 </joint>
@@ -174,5 +175,5 @@
     <origin xyz="0.0 0.0 0.0" rpy="0 0 0" />
     <mass value="0.3" />
-    <inertia ixx="0.1" ixy="0.1" ixz="0.1" iyy="0.1" iyz="0.1" izz="0.1"/>
+    <inertia ixx="0.119924" ixy="-0.0003874" ixz="-0.0010433" iyy="0.166674" iyz="5.8010177" izz="0.1314669"/>
 </inertial>
 <visual>
@@ -201,6 +202,6 @@
 <inertial>
     <origin xyz="0.0 0.0 0.0" rpy="0 0 0" />
-    <mass value="5" />
-    <inertia ixx="0.1" ixy="0.1" ixz="0.1" iyy="0.1" iyz="0.1" izz="0.1"/>
+    <mass value="0.5" />
+    <inertia ixx="0.10917" ixy="1.3005" ixz="-0.01020" iyy="0.15687" iyz="3.44815" izz="0.1"/>
 </inertial>
 <visual>
@@ -222,5 +223,5 @@
 <joint
     name="bum_zrj" type="revolute">
-    <origin xyz="-0.02 -0.265 0.16" rpy="0 0 0" />
+    <origin xyz="-0.02 -0.265 0.16" rpy="0 -0.3 0" />
     <parent link="base_body" />
     <child link="bum_zr" />
@@ -231,5 +232,5 @@
 <link name="bum_zr">
 <inertial>
-    <origin xyz="0.0 0.0 0.0" rpy="0 0 0" />
+    <origin xyz="0.0 0.0 -0.19" rpy="0 0 0" />
     <mass value="0.3" />
     <inertia ixx="0.1" ixy="0.1" ixz="0.1" iyy="0.1" iyz="0.1" izz="0.1"/>
@@ -259,5 +260,5 @@
 <link name="bum_xr">
 <inertial>
-    <origin xyz="0.0 0.0 0.0" rpy="0 0 0" />
+    <origin xyz="0.0 0.0 -0.19" rpy="0 0 0" />
     <mass value="0.3" />
     <inertia ixx="0.1" ixy="0.1" ixz="0.1" iyy="0.1" iyz="0.1" izz="0.1"/>
@@ -287,7 +288,7 @@
 <link name="right_hip">
 <inertial>
-    <origin xyz="0.0 0.0 0.0" rpy="0 0 0" />
-    <mass value="0.3" />
-    <inertia ixx="0.1" ixy="0.1" ixz="0.1" iyy="0.1" iyz="0.1" izz="0.1"/>
+    <origin xyz="0.0 0 -0.19" rpy="0 0 0" />
+    <mass value="0.3" />
+    <inertia ixx="0.31319" ixy="-1.5919" ixz="0.00039" iyy="0.314057" iyz="-0.00060" izz="0.02458"/>
 </inertial>
 <visual>
@@ -306,5 +307,5 @@
 <joint
     name="knee_right" type="revolute">
-    <origin xyz="0 0 -0.335" rpy="0 0 0" />
+    <origin xyz="0 0 -0.335" rpy="0 -0.5 0" />
     <parent link="right_hip" />
     <child link="right_shin" />
@@ -315,7 +316,7 @@
 <link name="right_shin">
 <inertial>
-    <origin xyz="0.0 0.0 0.0" rpy="0 0 0" />
-    <mass value="0.3" />
-    <inertia ixx="0.1" ixy="0.1" ixz="0.1" iyy="0.1" iyz="0.1" izz="0.1"/>
+    <origin xyz="0.0 0.0 -0.2" rpy="0 0 0" />
+    <mass value="0.3" />
+    <inertia ixx="0.283162" ixy="0.00034" ixz="0.001493" iyy="0.284290" iyz="0.000595" izz="0.0277465"/>
 </inertial>
 <visual>
@@ -334,9 +335,9 @@
 <joint
     name="ankle_rj" type="revolute">
-    <origin xyz="0 0 -0.58" rpy="0 0 0" />
+    <origin xyz="0 0 -0.58" rpy="0 0.3 0" />
     <parent link="right_shin" />
     <child link="right_ankle" />
     <axis xyz="0 1 0" />
-    <limit lower="-1.3" upper="0" effort="150.0" velocity="3"/>
+    <limit lower="-1.3" upper="0.3" effort="150.0" velocity="3"/>
     <!-- dynamics damping="5" friction="0.0"/ -->
 </joint>
@@ -345,5 +346,5 @@
     <origin xyz="0.0 0.0 0.0" rpy="0 0 0" />
     <mass value="0.3" />
-    <inertia ixx="0.1" ixy="0.1" ixz="0.1" iyy="0.1" iyz="0.1" izz="0.1"/>
+    <inertia ixx="0.119924" ixy="-0.0003874" ixz="-0.0010433" iyy="0.166674" iyz="5.8010177" izz="0.1314669"/>
 </inertial>
 <visual>
@@ -372,6 +373,6 @@
 <inertial>
     <origin xyz="0.0 0.0 0.0" rpy="0 0 0" />
-    <mass value="5" />
-    <inertia ixx="0.1" ixy="0.1" ixz="0.1" iyy="0.1" iyz="0.1" izz="0.1"/>
+    <mass value="0.5" />
+    <inertia ixx="0.119924" ixy="-0.0003874" ixz="-0.0010433" iyy="0.166674" iyz="5.8010177" izz="0.1314669"/>
 </inertial>
 <visual>
@@ -460,5 +461,5 @@
     <origin xyz="0.0 0.0 0.0" rpy="0 0 0" />
     <mass value="0.3" />
-    <inertia ixx="0.1" ixy="0.1" ixz="0.1" iyy="0.1" iyz="0.1" izz="0.1"/>
+    <inertia ixx="0.030306" ixy="1.072426" ixz="-0.00014" iyy="0.123799" iyz="-3.24634" izz="0.10389"/>
 </inertial>
 <visual>
@@ -488,5 +489,5 @@
     <origin xyz="0.0 0.0 0.0" rpy="0 0 0" />
     <mass value="0.3" />
-    <inertia ixx="0.1" ixy="0.1" ixz="0.1" iyy="0.1" iyz="0.1" izz="0.1"/>
+    <inertia ixx="0.37633" ixy="-5.2759" ixz="-8.13739" iyy="0.382769" iyz="-0.00136" izz="0.03977"/>
 </inertial>
 <visual>
@@ -575,5 +576,5 @@
     <origin xyz="0.0 0.0 0.0" rpy="0 0 0" />
     <mass value="0.3" />
-    <inertia ixx="0.1" ixy="0.1" ixz="0.1" iyy="0.1" iyz="0.1" izz="0.1"/>
+    <inertia ixx="0.030306" ixy="1.072426" ixz="-0.00014" iyy="0.123799" iyz="-3.24634" izz="0.10389"/>
 </inertial>
 <visual>
@@ -603,5 +604,5 @@
     <origin xyz="0.0 0.0 0.0" rpy="0 0 0" />
     <mass value="0.3" />
-    <inertia ixx="0.1" ixy="0.1" ixz="0.1" iyy="0.1" iyz="0.1" izz="0.1"/>
+    <inertia ixx="0.37633" ixy="-5.2759" ixz="-8.13739" iyy="0.382769" iyz="-0.00136" izz="0.03977"/>
 </inertial>
 <visual>

Commit message: controllers change but did not work on stable basis

File: catbot_description/urdf/bot.xacro (robot description, xacro)
@@ -218,4 +218,40 @@
 </collision>
 </link>
+<joint
+    name="contact_lj" type="fixed">
+    <origin xyz="0 0 -0.043" rpy="0 0 0" />
+    <parent link="left_foot" />
+    <child link="left_leg_contact_sensor" />
+    <axis xyz="0 1 0" />
+    <!-- <limit lower="-0.4" upper="0.7" effort="150.0" velocity="3"/> -->
+    <!-- dynamics damping="5" friction="0.0"/ -->
+</joint>
+<link name="left_leg_contact_sensor">
+<inertial >
+            <origin xyz="0 0 0" rpy="0 0 0"/>
+            <mass value="0.01" />
+            <inertia ixx="1.28e-06" ixy="0.0" ixz="0.0" iyy="1.28e-06" iyz="0.0" izz="1.28e-06"/>
+        </inertial>
+        <collision>
+            <origin xyz="0 0 0" rpy="0 0 0"/>
+            <geometry>
+                <!--
+                <sphere radius="0.030"/>
+                -->
+                <box size="0.01 0.01 0.01"/>
+                <!-- <sphere radius="0.01"/> -->
+            </geometry>
+        </collision>
+        <visual>
+            <origin rpy="0.0 0 0" xyz="0 0 0"/>
+            <geometry>
+                <!--
+                <sphere radius="0.030"/>
+                -->
+                <box size="0.01 0.01 0.01"/>
+                <!-- <sphere radius="0.01"/> -->
+            </geometry>
+        </visual>
+</link>
 <!-- ##########################################################
      ######################### right leg ########################
@@ -389,4 +425,40 @@
 </collision>
 </link>
+<joint
+    name="contact_rj" type="fixed">
+    <origin xyz="0 0 -0.043" rpy="0 0 0" />
+    <parent link="right_foot" />
+    <child link="right_leg_contact_sensor" />
+    <axis xyz="0 1 0" />
+    <!-- <limit lower="-" upper="0.7" effort="150.0" velocity="3"/> -->
+    <!-- dynamics damping="5" friction="0.0"/ -->
+</joint>
+<link name="right_leg_contact_sensor">
+<inertial >
+            <origin xyz="0 0 0" rpy="0 0 0"/>
+            <mass value="0.01" />
+            <inertia ixx="1.28e-06" ixy="0.0" ixz="0.0" iyy="1.28e-06" iyz="0.0" izz="1.28e-06"/>
+        </inertial>
+        <collision>
+            <origin xyz="0 0 0" rpy="0 0 0"/>
+            <geometry>
+                <!--
+                <sphere radius="0.030"/>
+                -->
+                <box size="0.01 0.01 0.01"/>
+                <!-- <sphere radius="0.01"/> -->
+            </geometry>
+        </collision>
+        <visual>
+            <origin rpy="0.0 0 0" xyz="0 0 0"/>
+            <geometry>
+                <!--
+                <sphere radius="0.030"/>
+                -->
+                <box size="0.01 0.01 0.01"/>
+                <!-- <sphere radius="0.01"/> -->
+            </geometry>
+        </visual>
+</link>
 <!-- ##########################################################
      ######################### right hand ########################

Commit message: joint pub rectified and controller connection script changed as per our robot. yet to be tested

File: catbot_description/urdf/bot.xacro (robot description, xacro)
@@ -55,5 +55,5 @@
     <child link="bum_zl" />
     <axis xyz="0 0 1" />
-    <limit lower="-0.345" upper="0.345" effort="150.0" velocity="3"/>
+    <limit lower="-0.345" upper="0.345" effort="1000" velocity="3"/>
     <!-- dynamics damping="5" friction="0.0"/ -->
 </joint>
@@ -83,5 +83,5 @@
     <child link="bum_xl" />
     <axis xyz="1 0 0" />
-    <limit lower="-0.345" upper="1" effort="150.0" velocity="3"/>
+    <limit lower="-0.345" upper="1" effort="1000" velocity="3"/>
     <!-- dynamics damping="5" friction="0.0"/ -->
 </joint>
@@ -112,5 +112,5 @@
     <child link="left_hip" />
     <axis xyz="0 1 0" />
-    <limit lower="0" upper="1" effort="150.0" velocity="3"/>
+    <limit lower="0" upper="1" effort="1000" velocity="3"/>
     <!-- dynamics damping="5" friction="0.0"/ -->
 </joint>
@@ -140,5 +140,5 @@
     <child link="left_shin" />
     <axis xyz="0 1 0" />
-    <limit lower="-1.3" upper="0" effort="150.0" velocity="3"/>
+    <limit lower="-1.3" upper="0" effort="1000" velocity="3"/>
     <!-- dynamics damping="5" friction="0.0"/ -->
 </joint>
@@ -168,5 +168,5 @@
     <child link="left_ankle" />
     <axis xyz="0 1 0" />
-    <limit lower="-1.3" upper="0.3" effort="150.0" velocity="3"/>
+    <limit lower="-1.3" upper="0.3" effort="1000" velocity="3"/>
     <!-- dynamics damping="5" friction="0.0"/ -->
 </joint>
@@ -196,5 +196,5 @@
     <child link="left_foot" />
     <axis xyz="0 1 0" />
-    <limit lower="-0.4" upper="0.7" effort="150.0" velocity="3"/>
+    <limit lower="-0.4" upper="0.7" effort="1000" velocity="3"/>
     <!-- dynamics damping="5" friction="0.0"/ -->
 </joint>
@@ -224,5 +224,5 @@
     <child link="left_leg_contact_sensor" />
     <axis xyz="0 1 0" />
-    <!-- <limit lower="-0.4" upper="0.7" effort="150.0" velocity="3"/> -->
+    <!-- <limit lower="-0.4" upper="0.7" effort="1000" velocity="3"/> -->
     <!-- dynamics damping="5" friction="0.0"/ -->
 </joint>
@@ -239,5 +239,5 @@
                 <sphere radius="0.030"/>
                 -->
-                <box size="0.01 0.01 0.01"/>
+                <box size="0.015 0.015 0.015"/>
                 <!-- <sphere radius="0.01"/> -->
             </geometry>
@@ -249,5 +249,5 @@
                 <sphere radius="0.030"/>
                 -->
-                <box size="0.01 0.01 0.01"/>
+                <box size="0.015 0.01 0.015"/>
                 <!-- <sphere radius="0.01"/> -->
             </geometry>
@@ -263,5 +263,5 @@
     <child link="bum_zr" />
     <axis xyz="0 0 1" />
-    <limit lower="-0.345" upper="0.345" effort="150.0" velocity="3"/>
+    <limit lower="-0.345" upper="0.345" effort="1000" velocity="3"/>
     <!-- dynamics damping="5" friction="0.0"/ -->
 </joint>
@@ -291,5 +291,5 @@
     <child link="bum_xr" />
     <axis xyz="1 0 0" />
-    <limit lower="-1" upper="0.345" effort="150.0" velocity="3"/>
+    <limit lower="-1" upper="0.345" effort="1000" velocity="3"/>
     <!-- dynamics damping="5" friction="0.0"/ -->
 </joint>
@@ -319,5 +319,5 @@
     <child link="right_hip" />
     <axis xyz="0 1 0" />
-    <limit lower="0" upper="1" effort="150.0" velocity="3"/>
+    <limit lower="0" upper="1" effort="1000" velocity="3"/>
     <!-- dynamics damping="5" friction="0.0"/ -->
 </joint>
@@ -347,5 +347,5 @@
     <child link="right_shin" />
     <axis xyz="0 1 0" />
-    <limit lower="-1.3" upper="0" effort="150.0" velocity="3"/>
+    <limit lower="-1.3" upper="0" effort="1000" velocity="3"/>
     <!-- dynamics damping="5" friction="0.0"/ -->
 </joint>
@@ -375,5 +375,5 @@
     <child link="right_ankle" />
     <axis xyz="0 1 0" />
-    <limit lower="-1.3" upper="0.3" effort="150.0" velocity="3"/>
+    <limit lower="-1.3" upper="0.3" effort="1000" velocity="3"/>
     <!-- dynamics damping="5" friction="0.0"/ -->
 </joint>
@@ -403,5 +403,5 @@
     <child link="right_foot" />
     <axis xyz="0 1 0" />
-    <limit lower="-0.4" upper="0.7" effort="150.0" velocity="3"/>
+    <limit lower="-0.4" upper="0.7" effort="1000" velocity="3"/>
     <!-- dynamics damping="5" friction="0.0"/ -->
 </joint>
@@ -431,5 +431,5 @@
     <child link="right_leg_contact_sensor" />
     <axis xyz="0 1 0" />
-    <!-- <limit lower="-" upper="0.7" effort="150.0" velocity="3"/> -->
+    <!-- <limit lower="-" upper="0.7" effort="1000" velocity="3"/> -->
     <!-- dynamics damping="5" friction="0.0"/ -->
 </joint>
@@ -446,5 +446,5 @@
                 <sphere radius="0.030"/>
                 -->
-                <box size="0.01 0.01 0.01"/>
+                <box size="0.015 0.015 0.015"/>
                 <!-- <sphere radius="0.01"/> -->
             </geometry>
@@ -456,5 +456,5 @@
                 <sphere radius="0.030"/>
                 -->
-                <box size="0.01 0.01 0.01"/>
+                <box size="0.015 0.015 0.015"/>
                 <!-- <sphere radius="0.01"/> -->
             </geometry>
@@ -470,5 +470,5 @@
     <child link="shoulder_zr" />
     <axis xyz="0 0 1" />
-    <limit lower="-0.345" upper="1.65" effort="150.0" velocity="3"/>
+    <limit lower="-0.345" upper="1.65" effort="1000" velocity="3"/>
     <!-- dynamics damping="5" friction="0.0"/ -->
 </joint>
@@ -498,5 +498,5 @@
     <child link="shoulder_xr" />
     <axis xyz="1 0 0" />
-    <limit lower="-0.1" upper="1.6" effort="150.0" velocity="3"/>
+    <limit lower="-0.1" upper="1.6" effort="1000" velocity="3"/>
     <!-- dynamics damping="5" friction="0.0"/ -->
 </joint>
@@ -526,5 +526,5 @@
     <child link="right_shoulder" />
     <axis xyz="0 1 0" />
-    <limit lower="0" upper="3" effort="150.0" velocity="3"/>
+    <limit lower="0" upper="3" effort="1000" velocity="3"/>
     <!-- dynamics damping="5" friction="0.0"/ -->
 </joint>
@@ -554,5 +554,5 @@
     <child link="right_forearm" />
     <axis xyz="1 0 0" />
-    <limit lower="-1.6" upper="0" effort="150.0" velocity="3"/>
+    <limit lower="-1.6" upper="0" effort="1000" velocity="3"/>
     <!-- dynamics damping="5" friction="0.0"/ -->
 </joint>
@@ -585,5 +585,5 @@
     <child link="shoulder_zl" />
     <axis xyz="0 0 1" />
-    <limit lower="-1.65" upper="0.1" effort="150.0" velocity="3"/>
+    <limit lower="-1.65" upper="0.1" effort="1000" velocity="3"/>
     <!-- dynamics damping="5" friction="0.0"/ -->
 </joint>
@@ -613,5 +613,5 @@
     <child link="shoulder_xl" />
     <axis xyz="1 0 0" />
-    <limit lower="-0.1" upper="1.6" effort="150.0" velocity="3"/>
+    <limit lower="-0.1" upper="1.6" effort="1000" velocity="3"/>
     <!-- dynamics damping="5" friction="0.0"/ -->
 </joint>
@@ -641,5 +641,5 @@
     <child link="left_shoulder" />
     <axis xyz="0 1 0" />
-    <limit lower="-3" upper="0" effort="150.0" velocity="3"/>
+    <limit lower="-3" upper="0" effort="1000" velocity="3"/>
     <!-- dynamics damping="5" friction="0.0"/ -->
 </joint>
@@ -669,5 +669,5 @@
     <child link="left_forearm" />
     <axis xyz="1 0 0" />
-    <limit lower="-1.6" upper="0" effort="150.0" velocity="3"/>
+    <limit lower="-1.6" upper="0" effort="1000" velocity="3"/>
     <!-- dynamics damping="5" friction="0.0"/ -->
 </joint>
